File: Business_Card_PCB-main/Masters_and_bs.kicad_pcb (KiCad board)
At the start: 2 copper layers, 86.6 x 54.7 mm, 24 parts, among them U1 NT3H1101W0FHKH

Commit message: added another v
added another version with the EE masters removed, using this for the career fair 2025/2026
Other:
- board text added: "Caleb J. Murray | Radar Engineer BS. Computer Engineering MS. Electrical Engineering Univ. Tennessee, 2027"
- board text removed: "Caleb J. Murray | Radar Engineer BS. Computer Engineering University Of Tennessee, 2027"
Changed lines of the file:
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@@
 			(at 0 1.55 90)
 			(layer "F.Fab")
-			(hide yes)
 			(effects
 				(font
@@
 			(layer "F.CrtYd")
 		)
+		(fp_text user "${REFERENCE}"
+			(at 0 -1.45 90)
+			(layer "F.Fab")
+			(effects
+				(font
+					(size 1 1)
+					(thickness 0.15)
+				)
+			)
+		)
 		(pad "1" smd circle
 			(at 0 0 90)
@@
 			(fill no)
 			(layer "F.CrtYd")
+			(net 1930368)
 		)
 		(pad "1" smd circle
@@
 			(layer "F.CrtYd")
 		)
+		(fp_text user "${REFERENCE}"
+			(at 0 -1.45 90)
+			(layer "F.Fab")
+			(effects
+				(font
+					(size 1 1)
+					(thickness 0.15)
+				)
+			)
+		)
 		(pad "1" smd circle
 			(at 0 0 90)
@@
 			(fill no)
 			(layer "F.CrtYd")
+			(net 1930368)
 		)
 		(pad "1" smd circle
@@
 			(fill no)
 			(layer "F.CrtYd")
+			(net 1930368)
 		)
 		(pad "1" smd circle
@@
 			(fill no)
 			(layer "F.CrtYd")
+			(net 1930368)
+		)
+		(fp_text user "${REFERENCE}"
+			(at 0 -1.45 90)
+			(layer "F.Fab")
+			(effects
+				(font
+					(size 1 1)
+					(thickness 0.15)
+				)
+			)
 		)
 		(pad "1" smd circle
@@
 		)
 	)
-	(gr_text "Caleb J. Murray | Radar Engineer\n\nBS. Computer Engineering\nUniversity Of Tennessee, 2027"
+	(gr_text "Caleb J. Murray | Radar Engineer\n\nBS. Computer Engineering\nMS. Electrical Engineering\nUniv. Tennessee, 2027"
 		(at 109.55 71.95 0)
 		(layer "F.Cu")
@@
 		)
 	)
-	(gr_text "Caleb J. Murray | Radar Engineer\n\nBS. Computer Engineering\nUniversity Of Tennessee, 2027"
+	(gr_text "Caleb J. Murray | Radar Engineer\n\nBS. Computer Engineering\nMS. Electrical Engineering\nUniv. Tennessee, 2027"
 		(at 109.55 71.95 0)
 		(layer "F.Mask")
